File: flight_controller_atlas/flight_controller_atlas.kicad_pcb (KiCad board)
At the start: 4 copper layers, 51.1 x 45 mm, 61 parts, among them J1 USB_B_Micro, J10 Screw_Terminal_01x02, J11 Screw_Terminal_01x02, J12 GND, J2 Ext 5v, J3 SM03B-SRSS-TB, J4 Screw_Terminal_01x02, J5 Screw_Terminal_01x02, J6 Screw_Terminal_01x02, J7 Screw_Terminal_01x02, J8 Screw_Terminal_01x02, J9 Screw_Terminal_01x02, Q1 DMP3099L, U1 RP2350A-QFN60, U2 ICM-20948, U3 LM3940IMPX-3.3_NOPB, U4 W25Q128JVS, U7 MIC5504-3.3YM5-TR, X1 ABM8-272-T3

Commit message: Add files via upload
v0.6 with barometer pt2
Parts:
- added C26: 100n, Capacitor_SMD:C_0402_1005Metric, F.Cu at (110.5, 90.7)
- added C27: 100n, Capacitor_SMD:C_0402_1005Metric, F.Cu at (115.7, 91.3)
- added R15: 4.7k, Resistor_SMD:R_0402_1005Metric, F.Cu at (111.0, 93.1)
- added R9: 4.7k, Resistor_SMD:R_0402_1005Metric, F.Cu at (115.7, 89.7)
- added U5: BMP384, custom_footprint:LGA10_2.0X2.0X0.95_BOS, F.Cu at (112.6, 90.7)
- D1: footprint LED_SMD:LED_0201_0603Metric -> custom_footprint:LED_CMD15-21_VCC
- moved D1 2.17 mm to (138.7, 74.3)
- moved R12 1.27 mm to (123.8, 71.0)
- moved R11 1.20 mm to (124.8, 71.0)
Connections:
- U1 pad 32: unconnected-(U1-GPIO20-Pad32) -> /SDA
- U1 pad 33: unconnected-(U1-GPIO21-Pad33) -> /SCL
Routing:
- net /SCL: track 0.00 -> 37.3 mm, vias 0 -> 2
- net /SDA: track 0.00 -> 34.2 mm, vias 0 -> 2
- net +3V3: track 108.3 -> 116.4 mm, vias 17 -> 21
- net GND: track 74.7 -> 81.2 mm, vias 29 -> 31
- net Net-(J10-Pin_2): track 27.8 -> 25.2 mm
- net Net-(D1-A): track 2.18 -> 3.45 mm
- net /+: track 31.3 -> 30.1 mm
- net /-: track 30.3 -> 29.2 mm
- net Net-(U1-USB_DM): track 5.09 -> 6.10 mm
- net Net-(J11-Pin_2): track 18.0 -> 18.6 mm
Other:
- board size 51.1 x 45 mm -> 51 x 45 mm
- board text added: "Baramoter"
- board text added: "IMU"
- board text added: "v0.6"
