File: flight_controller_atlas/flight_controller_atlas.kicad_sch (KiCad schematic)
At the start: 39 parts, among them J1 USB_B_Micro, J2 Ext 3.3v, Q1 DMP3099L, SW1 SW_Push, U1 RP2350A-QFN60, U2 ICM-20948, U3 LM3940IMPX-3.3_NOPB, U4 W25Q128JVS

Commit message: Add files via upload
Updated Schematic, v0.2
Parts:
- added C22, C23: 15p, symbol Device:C
- added J3: SM03B-SRSS-TB, CONN_SM03B-SRSS-TB_JST, symbol 2026-01-15_20-24-45:SM03B-SRSS-TB
- added J4: Screw_Terminal_01x09, symbol Connector:Screw_Terminal_01x09
- added R10: 1k, symbol Device:R_US
- added R11, R12: 27, symbol Device:R_US
- added X1: ABM8-272-T3, ABM8-272-T3_ABR, symbol 2026-01-15_19-57-48:ABM8-272-T3
Connections:
- net GND: now also C22.2, C23.2, J3.2, X1.2, X1.4
- net at U1.16 (GPIO12): now also J4.6 (Pin_6)
- net at U1.17 (GPIO13): now also J4.7 (Pin_7)
- net at U1.18 (GPIO14): now also J4.8 (Pin_8)
- net at U1.19 (GPIO15): now also J4.9 (Pin_9)
- net at U1.21 (XIN): now also C22.1, X1.1
- net at U1.22 (XOUT): now also R10.1
- net at U1.24 (SWCLK): now also J3.1
- net at U1.25 (SWDIO): now also J3.3
- net at U1.4 (GPIO2): now also J4.1 (Pin_1)
- net at U1.5 (GPIO3): now also J4.2 (Pin_2)
- net at U1.51 (USB_DM): now also R11.1; no longer J1.2 (D-)
- net at U1.52 (USB_DP): now also R12.1; no longer J1.3 (D+)
- net at U1.7 (GPIO4): now also J4.3 (Pin_3)
- net at U1.8 (GPIO5): now also J4.4 (Pin_4)
- net at U1.9 (GPIO6): now also J4.5 (Pin_5)
- new net: J1.2 (D-), R11.2
- new net: C23.1, R10.2, X1.3
- new net: J1.3 (D+), R12.2
Other:
- note added: "12MHz Crystal"
- note added: "JST Debug Connector"
- note added: "Radio Receiver & ESC Control Screw Terminal"
- moved on the sheet: C1, C10, C11, C12, C13, C14, C15, C16, C17, C18, C19, C2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

Commit message: Add files via upload
Atlas flight controller v0.4
Parts:
- removed J4: Screw_Terminal_01x09, symbol Connector:Screw_Terminal_01x09
- removed R3: 33, symbol Device:R
- removed R9: 1k, symbol Device:R_US
- removed SW1: SW_Push, symbol Switch:SW_Push
- added C24, C25: 1uF, Capacitor_SMD:C_0402_1005Metric, symbol Device:C
- added D1: LED, LED_SMD:LED_0201_0603Metric, symbol Device:LED
- added FL1: BLM15AX601SN1D, custom_footprint:BEADC1005X55N, symbol BLM15AX601SN1D:BLM15AX601SN1D
- added J10, J11, J4, J5, J6, J7, J8, J9: Screw_Terminal_01x02, custom_footprint:691137710002, symbol Connector:Screw_Terminal_01x02
- added J12: GND, Connector_Wire:SolderWirePad_1x01_SMD_1x2mm, symbol Connector_Generic:Conn_01x01
- added R13: 330, Resistor_SMD:R_0402_1005Metric, symbol Device:R_US
- added R14: 33, Resistor_SMD:R_0402_1005Metric, symbol Device:R_US
- added R3: 1k, Resistor_SMD:R_0402_1005Metric, symbol Device:R_US
- added S1: TL3365AF180QG, custom_footprint:SW_TL3365AF180QG, symbol TL3365AF180QG:TL3365AF180QG
- added U7: MIC5504-3.3YM5-TR, custom_footprint:SOT-23-5_MC_MCH, symbol 2026-01-21_20-29-49:MIC5504-3.3YM5-TR
- C1, C10, C11, C12, C13, C14, C15, C16, C17, C18, C19, C2, C20, C21, C22, C23, C3, C4, C5, C6, C7, C8, C9: footprint (none) -> Capacitor_SMD:C_0402_1005Metric
- J1: footprint (none) -> custom_footprint:AMPHENOL_10118192-0001LF
- J2: value Ext 3.3v -> Ext 5v; footprint (none) -> Connector_Wire:SolderWirePad_1x01_SMD_1x2mm
- J3: footprint CONN_SM03B-SRSS-TB_JST -> custom_footprint:CONN_SM03B-SRSS-TB_JST
- L1: footprint (none) -> Inductor_SMD:L_Cenker_CKCS201610
- R1, R10, R11, R12, R2, R4, R5, R6, R7, R8: footprint (none) -> Resistor_SMD:R_0402_1005Metric
- U1: footprint (none) -> custom_footprint:RP2350A_QFN-60_EP_7.75x7.75_Pitch0.4mm
- U2: footprint Sensor_Motion:InvenSense_QFN-24_3x3mm_P0.4mm -> custom_footprint:QFN40P300X300X105-24N
- U3: footprint LM3940IMPX-3.3_NOPB:SOT230P700X180-4N -> custom_footprint:SOT230P700X180-4N
- X1: footprint ABM8-272-T3_ABR -> custom_footprint:ABM8-272-T3_ABR
Connections:
- net +3V3: now also U1.2 (GPIO0), U1.60 (QSPI_SS), U2.24 (SDA/SDI), U4.1 (~{CS}), FL1.2, R13.2, R14.1, R3.1; no longer U2.13 (VDD)
- net GND: now also C24.2, C25.2, D1.1 (K), J12.1 (Pin_1), S1.1, S1.2, U7.2 (GND); no longer U1.23 (DVDD), U1.39 (DVDD), U1.6 (DVDD)
- net at Q1.2 (S): now also C25.1, U7.5 (VOUT); no longer J2.1 (Pin_1)
- net at C7.1, U1.46 (VREG_AVDD): now also R14.2
- net -: now reaches J1.2 (D-), R11.2
- net at C18.1, C19.1, C20.1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: now also U1.23 (DVDD), U1.39 (DVDD), U1.6 (DVDD)
- net at U1.10 (GPIO7): now also J7.2 (Pin_2)
- net at U1.12 (GPIO8): now also J8.1 (Pin_1)
- net at U1.13 (GPIO9): now also J8.2 (Pin_2)
- net at U1.14 (GPIO10): now also J9.1 (Pin_1)
- net at U1.15 (GPIO11): now also J9.2 (Pin_2)
- net at U1.16 (GPIO12): now also J5.1 (Pin_1)
- net at U1.17 (GPIO13): now also J5.2 (Pin_2)
- net at U1.18 (GPIO14): now also J11.1 (Pin_1)
- net at U1.19 (GPIO15): now also J11.2 (Pin_2)
- net at U1.36 (GPIO24): now also J10.1 (Pin_1)
- net at U1.37 (GPIO25): now also J10.2 (Pin_2)
- net at U1.4 (GPIO2): now also J6.1 (Pin_1)
- net at U1.5 (GPIO3): now also J6.2 (Pin_2)
- net at U1.7 (GPIO4): now also J4.1 (Pin_1)
- net at U1.8 (GPIO5): now also J4.2 (Pin_2)
- net at U1.9 (GPIO6): now also J7.1 (Pin_1)
- net +: now reaches J1.3 (D+), R12.2
- new net: R3.2, S1.3, S1.4
- new net: C24.1, J2.1 (Pin_1), U7.1 (VIN)
- new net: D1.2 (A), R13.1
- new net: FL1.1, U2.13 (VDD)
Other:
- note added: "CH0"
- note added: "CH11"
- note added: "ESC Control Screw Terminal"
- note added: "Radio Reciever Channels"
- note added: "bootsel"
- note added: "decoupling capacitors (required for rp2350, one per IOVDD/DVDD pin)"
- note added: "primary flash 16MB"
- note removed: "Radio Receiver & ESC Control Screw Terminal"
- note removed: "decoupling capacitors (required for rp2350)"
- note removed: "primary flash"
- moved on the sheet: J2

Commit message: Add files via upload
v0.6 with barometer pt2
Parts:
- added C26, C27: 100n, Capacitor_SMD:C_0402_1005Metric, symbol Device:C
- added R15, R9: 4.7k, Resistor_SMD:R_0402_1005Metric, symbol Device:R_US
- added U5: BMP384, custom_footprint:LGA10_2.0X2.0X0.95_BOS, symbol 2026-01-23_15-50-37:BMP384
- D1: footprint LED_SMD:LED_0201_0603Metric -> custom_footprint:LED_CMD15-21_VCC
Connections:
- net +3V3: now also C26.1, C27.1, R15.2, R9.2, U5.1 (VDDIO), U5.10 (VDD), U5.5 (SDO), U5.6 (CSB)
- net GND: now also C26.2, C27.2, U5.3 (VSS), U5.8 (VSS), U5.9 (VSS)
- net SDA: now reaches U1.32 (GPIO20)
- net SDA: now also R9.1, U5.4 (SDI)
- net SCL: now reaches U1.33 (GPIO21)
- net SCL: now also R15.1, U5.2 (SCK)
Other:
- note added: "Barometer Sensor"
- note added: "I2C address: 0x77"
